File: ESP-Now-Gateway.kicad_sch (KiCad schematic)
At the start: 47 parts, among them J1 HR911105A, J2 PROG, J4 External GPIO Header, J5 Power Header, Q1 SS8050_C2150, Q2 SS8050_C2150, U1 AMS1117-3.3, U2 ESP32-WROOM-32, U3 LAN8720A, U4 CH343G

Commit message: Improve layout
Parts:
- R19, R20: footprint Resistor_SMD:R_0402_1005Metric -> Resistor_SMD:R_0603_1608Metric; LCSC Part # C25744 -> (none)
Changed lines of the file:
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@@
 			)
 		)
-		(property "Footprint" "Resistor_SMD:R_0402_1005Metric"
+		(property "Footprint" "Resistor_SMD:R_0603_1608Metric"
 			(at 105.41 55.118 90)
 			(effects
@@
 			)
 		)
-		(property "LCSC Part #" "C25744"
+		(property "LCSC Part #" ""
 			(at 105.41 53.34 0)
 			(effects
@@
 			)
 		)
-		(property "Footprint" "Resistor_SMD:R_0402_1005Metric"
+		(property "Footprint" "Resistor_SMD:R_0603_1608Metric"
 			(at 105.41 47.498 90)
 			(effects
@@
 			)
 		)
-		(property "LCSC Part #" "C25744"
+		(property "LCSC Part #" ""
 			(at 105.41 45.72 0)
 			(effects
