File: ESP-Now-Gateway.kicad_pcb (KiCad board)
At the start: 2 copper layers, 32 x 58.8 mm, 47 parts, among them J1 HR911105A, J2 PROG, J4 External GPIO Header, J5 Power Header, Q1 SS8050_C2150, Q2 SS8050_C2150, U1 AMS1117-3.3, U2 ESP32-WROOM-32, U3 LAN8720A, U4 CH343G

Commit message: Finalize pcb design
Parts:
- moved R5 2.47 mm to (116.7, 103.3), turned to 180 degrees
- moved C12 2.21 mm to (110.5, 70.5), turned to 0 degrees
- moved R2 1.92 mm to (123.2, 102.1)
- moved R4 1.57 mm to (126.3, 102.6)
- moved C14 1.26 mm to (110.5, 73.7)
- moved R7 1.25 mm to (110.5, 72.1)
- moved J4 0.75 mm to (106.8, 77.9)
- moved C3 0.60 mm to (110.5, 69.0)
- moved L1 0.60 mm to (120.8, 97.4)
- moved C5 0.56 mm to (103.7, 105.3)
- moved R6 0.56 mm to (131.8, 85.8)
- moved R15 0.44 mm to (114.6, 95.8)
- moved R19 0.44 mm to (114.6, 94.8)
- moved C1 0.34 mm to (104.8, 96.9)
- moved C4 0.31 mm to (111.2, 66.5)
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Routing:
- net VBUS: track 52.8 -> 58.1 mm
- net +3V3: track 157.5 -> 153.1 mm
- net Net-(J1-Pad10): track 17.4 -> 19.6 mm, vias 0 -> 1
- net /ETH_TXEN: track 32.6 -> 30.7 mm
- net /ETH_MDC: track 33.7 -> 31.9 mm
- net GND: track 37.4 -> 35.6 mm, vias 238 -> 219
- net /PHY_RXER: track 20.6 -> 18.8 mm
- net /ESP_IO14: track 10.3 -> 12.1 mm
- net /ETH_RXD0: track 24.7 -> 23.0 mm
- net /ETH_TXD1: track 36.7 -> 35.1 mm
- net /PHY_L2: track 19.1 -> 17.5 mm
- net /ESP_SENSOR_VN_IO39: track 14.8 -> 16.3 mm
- net /ETH_TXD0: track 31.0 -> 29.5 mm
- net /ESP_IO35: track 19.3 -> 20.5 mm
- net /BOOT0: track 45.3 -> 44.1 mm
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Other:
- board text added: "EN"
- board text added: "IO0"
- board text added: "IO13 - IO12"
- board text added: "IO15 - IO2"
- board text added: "IO33 - IO5"
- board text added: "IO34 - IO36"
- board text added: "IO35 - IO39"
- board text added: "IO4 - IO14"
- board text added: "Input Only: - IO34 - IO35 - IO39 - IO36 Strapping: - IO2 - IO5 - IO12 - IO14 - IO15 Normal: - IO4 - IO13 - IO33"
- board text added: "RX"
- board text added: "TX"

Commit message: Improve routing
Parts:
- moved C10 1.93 mm to (129.4, 98.1), turned to -90 degrees
- moved C8 1.89 mm to (131.0, 98.1), turned to -90 degrees
- moved R1 1.86 mm to (125.5, 99.7)
- moved R11 1.83 mm to (128.0, 99.4), turned to -90 degrees
- moved C11 1.55 mm to (120.5, 95.0)
- moved R12 1.47 mm to (120.5, 93.5)
- moved R14 1.44 mm to (132.1, 104.0), turned to 0 degrees
- moved R4 1.15 mm to (127.2, 101.8)
- moved R2 1.02 mm to (124.1, 101.8)
- moved R3 0.78 mm to (124.1, 104.0)
- moved C9 0.65 mm to (130.4, 92.2)
- moved R9 0.37 mm to (129.3, 91.2)
- moved C7 0.36 mm to (125.5, 90.7)
- moved R8 0.16 mm to (128.2, 90.1)
Routing:
- net /TX: track 80.5 -> 89.3 mm, vias 4 -> 5
- net GND: track 35.6 -> 27.3 mm, vias 219 -> 247
- net /BOOT0: track 44.1 -> 51.4 mm, vias 2 -> 4
- net /RX: track 80.9 -> 87.7 mm, vias 2 -> 5
- net /PHY_INT: track 28.2 -> 33.1 mm, vias 0 -> 4
- net /ESP_SENSOR_VN_IO39: track 16.3 -> 12.9 mm
- net /ESP_SENSOR_VP_IO36: track 12.3 -> 9.14 mm
- net /ETH_MDIO: track 26.5 -> 23.8 mm
- net /ESP_IO35: track 20.5 -> 17.9 mm
- net +3V3: track 153.1 -> 155.1 mm
- net /ETH_RXD1: track 25.3 -> 27.1 mm, vias 2 -> 4
- net /ESP_IO2: track 36.2 -> 38.0 mm, vias 2 -> 4
- net /PHY_L2: track 17.5 -> 18.9 mm
- net /TX+: track 14.8 -> 16.2 mm
- net /TX-: track 12.7 -> 11.5 mm
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
Commit message: More improvements for pcb
Parts:
- moved L1 1.41 mm to (122.1, 97.8)
Routing:
- net Net-(U3-VDD1A): track 12.7 -> 11.2 mm
- net /ESP_IO2: track 38.0 -> 37.4 mm

Commit message: More cleanup
Routing:
- net +3V3: track 155.5 -> 156.5 mm

Commit message: Improve layout
Parts:
- R19, R20: footprint Resistor_SMD:R_0402_1005Metric -> Resistor_SMD:R_0603_1608Metric
- moved R15 6.81 mm to (120.0, 100.0), turned to 90 degrees
- moved R5 4.54 mm to (121.0, 101.8)
- moved R16 1.72 mm to (114.5, 102.2), turned to 90 degrees
- moved Q1 1.47 mm to (117.3, 98.3)
- moved Q2 1.35 mm to (117.3, 101.8), turned to 0 degrees
- moved U4 0.40 mm to (109.4, 110.0)
- moved R19 0.36 mm to (114.7, 94.5)
- moved R3 0.15 mm to (124.2, 104.1)
- moved R1 0.10 mm to (125.5, 99.5)
- moved R20 0.09 mm to (103.2, 109.7)
Routing:
- net +3V3: track 156.5 -> 170.2 mm
- net GND: track 27.3 -> 38.4 mm, vias 247 -> 241
- net /BOOT0: track 51.4 -> 57.9 mm
- net /PHY_L2: track 19.1 -> 14.0 mm
- net /DTR: track 18.4 -> 22.6 mm
- net /RTS: track 14.4 -> 10.9 mm
- net Net-(Q1-B): track 1.66 -> 4.90 mm
- net Net-(Q2-B): track 4.64 -> 1.84 mm
- net /ETH_RXD0: track 22.4 -> 23.9 mm
- net /EN: track 38.1 -> 36.7 mm
- net /PHY_L1: track 12.3 -> 13.6 mm
- net /ETH_CRS_DV: track 14.7 -> 15.9 mm
- net /ESP_SENSOR_VP_IO36: track 9.14 -> 10.0 mm
- net /RX+: track 15.0 -> 14.2 mm
- net Net-(J1-Pad10): track 19.6 -> 20.3 mm, vias 1 -> 0
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
Commit message: Should be production ready
Other:
- board text added: "JLCJLCJLCJLC"
Changed lines of the file:
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@@
 		(sheetname "Root")
 		(sheetfile "ESP-Now-Gateway.kicad_sch")
-		(attr through_hole)
+		(attr through_hole exclude_from_pos_files exclude_from_bom)
 		(fp_line
 			(start -1.33 -1.33)
@@
 		(sheetname "Root")
 		(sheetfile "ESP-Now-Gateway.kicad_sch")
-		(attr through_hole)
+		(attr through_hole exclude_from_pos_files exclude_from_bom)
 		(fp_line
 			(start 3.87 -1.33)
@@
 		(sheetname "Root")
 		(sheetfile "ESP-Now-Gateway.kicad_sch")
-		(attr through_hole)
+		(attr through_hole exclude_from_pos_files exclude_from_bom)
 		(fp_line
 			(start -1.33 -1.33)
@@
 		)
 	)
+	(gr_text "JLCJLCJLCJLC"
+		(at 118.225 67.15 0)
+		(layer "F.SilkS")
+		(effects
+			(font
+				(size 1 1)
+				(thickness 0.2)
+				(bold yes)
+			)
+			(justify left bottom)
+		)
+	)
 	(segment
 		(start 106.67 97.42)
@@
 		(name "$teardrop_padvia$")
 		(hatch full 0.1)
-		(priority 30000)
+		(priority 30002)
 		(attr
 			(teardrop
@@
 		(polygon
 			(pts
-				(xy 104.507538 101.888909) (xy 104.861091 102.242462) (xy 105.532843 101.782843) (xy 105.250707 101.499293)
-				(xy 104.967157 101.217157)
+				(xy 104.45 101.25) (xy 104.45 101.75) (xy 105.25 101.9) (xy 105.251 101.5) (xy 105.25 101.1)
 			)
 		)
@@
 		(name "$teardrop_padvia$")
 		(hatch full 0.1)
-		(priority 30005)
+		(priority 30004)
 		(attr
 			(teardrop
@@
 		(polygon
 			(pts
-				(xy 104.25 101.75) (xy 104.25 101.25) (xy 103.880448 101.653073) (xy 104.249 101.5) (xy 103.880448 101.653073)
+				(xy 104 102.3) (xy 104.5 102.3) (xy 104.65 101.5) (xy 104.25 101.499) (xy 103.85 101.5)
 			)
 		)
@@
 		(name "$teardrop_padvia$")
 		(hatch full 0.1)
-		(priority 30003)
+		(priority 30005)
 		(attr
 			(teardrop
@@
 		(polygon
 			(pts
-				(xy 104.05 101.75) (xy 104.05 101.25) (xy 103.25 101.1) (xy 103.249 101.5) (xy 103.25 101.9)
+				(xy 104.25 101.75) (xy 104.25 101.25) (xy 103.880448 101.653073) (xy 104.249 101.5) (xy 103.880448 101.653073)
 			)
 		)
@@
 		(name "$teardrop_padvia$")
 		(hatch full 0.1)
-		(priority 30002)
+		(priority 30003)
 		(attr
 			(teardrop
@@
 		(polygon
 			(pts
-				(xy 104.45 101.25) (xy 104.45 101.75) (xy 105.25 101.9) (xy 105.251 101.5) (xy 105.25 101.1)
+				(xy 104.05 101.75) (xy 104.05 101.25) (xy 103.25 101.1) (xy 103.249 101.5) (xy 103.25 101.9)
 			)
 		)
@@
 		(name "$teardrop_padvia$")
 		(hatch full 0.1)
-		(priority 30004)
+		(priority 30000)
 		(attr
 			(teardrop
@@
 		(polygon
 			(pts
-				(xy 104 102.3) (xy 104.5 102.3) (xy 104.65 101.5) (xy 104.25 101.499) (xy 103.85 101.5)
+				(xy 104.507538 101.888909) (xy 104.861091 102.242462) (xy 105.532843 101.782843) (xy 105.250707 101.499293)
+				(xy 104.967157 101.217157)
 			)
 		)
@@
 		(name "$teardrop_padvia$")
 		(hatch full 0.1)
-		(priority 30005)
+		(priority 30006)
 		(attr
 			(teardrop
@@
 		(polygon
 			(pts
-				(xy 103.891064 100.737511) (xy 103.537511 101.091064) (xy 103.880448 101.653073) (xy 104.250707 101.500707)
-				(xy 104.532843 101.217157)
+				(xy 104.745593 101.03204) (xy 104.39204 101.385593) (xy 104.967157 101.782843) (xy 105.250707 101.500707)
+				(xy 105.25 101.1)
 			)
 		)
@@
 		(name "$teardrop_padvia$")
 		(hatch full 0.1)
-		(priority 30002)
+		(priority 30004)
 		(attr
 			(teardrop
@@
 		(polygon
 			(pts
-				(xy 104.05 101.75) (xy 104.05 101.25) (xy 103.25 101.1) (xy 103.249 101.5) (xy 103.25 101.9)
+				(xy 104.45 101.25) (xy 104.45 101.75) (xy 105.25 101.9) (xy 105.251 101.5) (xy 105.25 101.1)
 			)
 		)
@@
 		(name "$teardrop_padvia$")
 		(hatch full 0.1)
-		(priority 30004)
+		(priority 30001)
 		(attr
 			(teardrop
@@
 		(polygon
 			(pts
-				(xy 104.45 101.25) (xy 104.45 101.75) (xy 105.25 101.9) (xy 105.251 101.5) (xy 105.25 101.1)
+				(xy 103.45 101.25) (xy 103.45 101.75) (xy 104.25 101.9) (xy 104.251 101.5) (xy 104.25 101.1)
 			)
 		)
@@
 		(name "$teardrop_padvia$")
 		(hatch full 0.1)
-		(priority 30000)
+		(priority 30005)
 		(attr
 			(teardrop
@@
 		(polygon
 			(pts
-				(xy 103.5 100.7) (xy 103 100.7) (xy 102.85 101.5) (xy 103.25 101.501) (xy 103.65 101.5)
+				(xy 103.891064 100.737511) (xy 103.537511 101.091064) (xy 103.880448 101.653073) (xy 104.250707 101.500707)
+				(xy 104.532843 101.217157)
 			)
 		)
@@
 		(name "$teardrop_padvia$")
 		(hatch full 0.1)
-		(priority 30006)
+		(priority 30000)
 		(attr
 			(teardrop
@@
 		(polygon
 			(pts
-				(xy 104.745593 101.03204) (xy 104.39204 101.385593) (xy 104.967157 101.782843) (xy 105.250707 101.500707)
-				(xy 105.25 101.1)
+				(xy 103.5 100.7) (xy 103 100.7) (xy 102.85 101.5) (xy 103.25 101.501) (xy 103.65 101.5)
 			)
 		)
@@
 		(name "$teardrop_padvia$")
 		(hatch full 0.1)
-		(priority 30001)
+		(priority 30002)
 		(attr
 			(teardrop
@@
 		(polygon
 			(pts
-				(xy 103.45 101.25) (xy 103.45 101.75) (xy 104.25 101.9) (xy 104.251 101.5) (xy 104.25 101.1)
+				(xy 104.05 101.75) (xy 104.05 101.25) (xy 103.25 101.1) (xy 103.249 101.5) (xy 103.25 101.9)
 			)
 		)
